File: PCB/High-Altitude-Sync-Board/High-Altitude-Sync-Board.kicad_sch (KiCad schematic)
At the start: 65 parts, among them J1 USB_C_Receptacle_USB2.0_14P, J10 M80-9110099, J11 M80-9110099, J12 M80-9110099, J13 M80-9110099, J14 M80-9110099, J16 M80-4151098, J17 VN100T-UPDATE, J18 Conn_01x02, J19 Conn_01x02, J2 UBLOX_TRIGGER, J20 EXT_SYNC, J21 HR10A-7P-6S(73), J22 HR10A-7P-6S(73), J23 Conn_01x04, J24 SWD, J25 Conn_01x04, J26 UART, J3 M80-9110099, J4 M80-9110099, J5 M80-9110099, J6 M80-9110099, J7 VN100_T_CONN, J8 M80-9110099, J9 GHR-10V-S, U1 SN74AXC8T245PWR, U2 FT232RL, U3 LP5912-3.3DRV, U4 STM32L011F3Ux, X1 ECS-2520MV

Commit message: High Altitude Sync Board - V1
Parts:
- removed C8: 100nF, Capacitor_SMD:C_0603_1608Metric, symbol Device:C
- added J15, J27, J28, J29, J30, J31, J32, J33, J34, J35, J38, J39, J40, J41, J42, J43, J44, J45, J47, J48, J49, J51, J52, J54, J55, J57: MINI-SSHL, symbol Connector_Generic:Conn_01x01
- added J36, J37: GHR-04V-S, symbol Connector_Generic:Conn_01x04
- added J46, J50, J53, J56: GHR-02V-S, symbol Connector_Generic:Conn_01x02
- added TP1: 5V TP, TestPoint:TestPoint_THTPad_1.0x1.0mm_Drill0.5mm, symbol Connector:TestPoint
- added TP2: GND TP, TestPoint:TestPoint_THTPad_1.0x1.0mm_Drill0.5mm, symbol Connector:TestPoint
- added TP3: 3V3 TP, TestPoint:TestPoint_THTPad_1.0x1.0mm_Drill0.5mm, symbol Connector:TestPoint
- C1, C5, C7: digikey# (none) -> 311-1088-2-ND; manf# CC0603ZRY5V9BB104 -> CC0603KRX7R7BB104; mouser# (none) -> 603-CC603KRX7R7BB104
- C2, C3: digikey# (none) -> 311-1088-2-ND; manf# (none) -> CC0603KRX7R7BB104; mouser# (none) -> 603-CC603KRX7R7BB104
- J1: digikey# (none) -> 2073-USB4085-GF-ATR-ND; manf# (none) -> USB4085-GF-A
- J10, J11, J12, J13, J14, J5, J6, J8: value M80-9110099 -> M80; footprint (none) -> ~; digikey# (none) -> 952-2981-ND; manf# (none) -> M80-9110099
- J16: digikey# (none) -> 952-3724-ND; manf# (none) -> M80-4151098
- J17, J26: DNP (none) -> DNP; now not fitted
- J18, J19: value Conn_01x02 -> BM02B-GHS-TBT; digikey# (none) -> 455-BM02B-GHS-TBTTR-ND; manf# (none) -> BM02B-GHS-TBT
- J2: value UBLOX_TRIGGER -> SM02B-GHS-TB; digikey# (none) -> 455-1564-2-ND; manf# (none) -> SM02B-GHS-TB
- J20: value EXT_SYNC -> SM02B-GHS-TB; digikey# (none) -> 455-1564-2-ND; manf# (none) -> SM02B-GHS-TB
- J21, J22: digikey# (none) -> HR1588-ND; manf# (none) -> HR10A-7P-6S(73)
- J23, J25: value Conn_01x04 -> BM04B-GHS-TBT; digikey# (none) -> 455-BM04B-GHS-TBTTR-ND; manf# (none) -> BM04B-GHS-TBT
- J24: now not fitted
- J3, J4: value M80-9110099 -> M80; digikey# (none) -> 952-2981-ND; manf# (none) -> M80-9110099
- J7: digikey# (none) -> 455-SM10B-GHS-TBTR-ND; manf# (none) -> SM10B-GHS-TB
- J9: digikey# (none) -> 455-1600-ND; manf# (none) -> GHR-10V-S
- R1, R2: digikey# (none) -> CRCW06035K10FKEA; manf# (none) -> CRCW06035K10FKEA; mouser# (none) -> 71-CRCW0603-5.1K-E3
- R11, R12, R13, R14, R15, R16, R20, R21, R8, R9: value DNP -> 0R; DNP (none) -> DNP; digikey# (none) -> 311-0.0GRTR-ND; manf# (none) -> RC0603JR-070RL; mouser# (none) -> 603-RC0603JR-070RL; now not fitted
- R19, R22, R3, R4, R5, R6, R7: digikey# (none) -> 311-0.0GRTR-ND; manf# (none) -> RC0603JR-070RL; mouser# (none) -> 603-RC0603JR-070RL
- U1: digikey# (none) -> 296-48831-2-ND; manf# (none) -> SN74AXC8T245PWR
- U2: digikey# 768-1007-6-ND -> 768-FT232RNL-REELTR-ND; manf# FT232RL -> FT232RNL-REEL
- U3: digikey# (none) -> 296-47214-2-ND; manf# (none) -> LP5912-3.3DRVR
- U4: digikey# (none) -> 497-18800-2-ND; manf# (none) -> STM32L011F3U6TR
- X1: digikey# (none) -> XC2752TR; manf# (none) -> ECS-2520MV-250-CN-TR
Connections:
- net +3V3: now also C7.1, TP3.1
- net +5V: now also TP1.1
- net GND: now also TP2.1
- net at J11.1 (Pin_1): now also J16.4 (Pin_4); no longer J9.4 (Pin_4)
- net at J9.8 (Pin_8): now also J28.1 (Pin_1); no longer J5.1 (Pin_1)
- net at U2.17 (3V3OUT): no longer C7.1
- net at J3.1 (Pin_1): now also J16.10 (Pin_10); no longer J9.10 (Pin_10)
- net at J10.1 (Pin_1): now also J16.5 (Pin_5); no longer J9.5 (Pin_5)
- net at J16.1 (Pin_1): now also J14.1 (Pin_1)
- net at J16.2 (Pin_2): now also J13.1 (Pin_1)
- net at J16.3 (Pin_3): now also J12.1 (Pin_1)
- net at J16.6 (Pin_6): now also J8.1 (Pin_1)
- net at J16.7 (Pin_7): now also J6.1 (Pin_1)
- net at J16.8 (Pin_8): now also J5.1 (Pin_1)
- net at J16.9 (Pin_9): now also J4.1 (Pin_1)
- net at J9.2 (Pin_2): now also J34.1 (Pin_1); no longer J13.1 (Pin_1)
- net at J9.1 (Pin_1): now also J35.1 (Pin_1); no longer J14.1 (Pin_1)
- net at J9.3 (Pin_3): now also J33.1 (Pin_1); no longer J12.1 (Pin_1)
- net at J9.6 (Pin_6): now also J30.1 (Pin_1); no longer J8.1 (Pin_1)
- net at J9.7 (Pin_7): now also J29.1 (Pin_1); no longer J6.1 (Pin_1)
- net at J9.9 (Pin_9): now also J27.1 (Pin_1); no longer J4.1 (Pin_1)
- new net: J37.4 (Pin_4), J42.1 (Pin_1)
- new net: J49.1 (Pin_1), J50.1 (Pin_1)
- new net: J55.1 (Pin_1), J56.1 (Pin_1)
- new net: J50.2 (Pin_2), J51.1 (Pin_1)
- new net: J53.2 (Pin_2), J54.1 (Pin_1)
- new net: J36.3 (Pin_3), J39.1 (Pin_1)
- new net: J37.2 (Pin_2), J44.1 (Pin_1)
- new net: J15.1 (Pin_1), J9.10 (Pin_10)
- new net: J32.1 (Pin_1), J9.4 (Pin_4)
- new net: J36.1 (Pin_1), J41.1 (Pin_1)
- new net: J36.2 (Pin_2), J40.1 (Pin_1)
- new net: J36.4 (Pin_4), J38.1 (Pin_1)
- new net: J56.2 (Pin_2), J57.1 (Pin_1)
- new net: J37.3 (Pin_3), J43.1 (Pin_1)
- new net: J31.1 (Pin_1), J9.5 (Pin_5)
- new net: J52.1 (Pin_1), J53.1 (Pin_1)
- new net: J46.2 (Pin_2), J48.1 (Pin_1)
- new net: J46.1 (Pin_1), J47.1 (Pin_1)
- new net: J37.1 (Pin_1), J45.1 (Pin_1)
- no-connect marks 43 -> 34
Other:
- note added: "This corresponds to the JST conn and and crimps"
- moved on the sheet: C1, C10, C4, C6, D1, D2, J1, J16, J18, J19, J2, J20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
